File: ErgoDOX.sch (KiCad schematic (older format))
At the start: 101 parts, among them J1 USB, J2 3.5mm, J3 JMP, J4 JMP, SW1 SWITCH_PUSH, SW10 SWITCH_PUSH, SW11 SWITCH_PUSH, SW12 SWITCH_PUSH, SW13 SWITCH_PUSH, SW14 SWITCH_PUSH, SW15 SWITCH_PUSH, SW16 SWITCH_PUSH, SW17 SWITCH_PUSH, SW18 SWITCH_PUSH, SW19 SWITCH_PUSH, SW2 SWITCH_PUSH, SW20 SWITCH_PUSH, SW21 SWITCH_PUSH, SW22 SWITCH_PUSH, SW23 SWITCH_PUSH, SW24 SWITCH_PUSH, SW25 SWITCH_PUSH, SW26 SWITCH_PUSH, SW27 SWITCH_PUSH, SW28 SWITCH_PUSH, SW29 SWITCH_PUSH, SW3 SWITCH_PUSH, SW30 SWITCH_PUSH, SW31 SWITCH_PUSH, SW32 SWITCH_PUSH, SW33 SWITCH_PUSH, SW34 SWITCH_PUSH, SW35 SWITCH_PUSH, SW36 SWITCH_PUSH, SW37 SWITCH_PUSH, SW38 SWITCH_PUSH, SW39 SWITCH_PUSH, SW4 SWITCH_PUSH, SW40 SWITCH_PUSH, SW41 SWITCH_PUSH, SW42 SWITCH_PUSH, SW43 SWITCH_PUSH, SW44 SWITCH_PUSH, SW5 SWITCH_PUSH, SW6 SWITCH_PUSH, SW7 SWITCH_PUSH, SW8 SWITCH_PUSH, SW9 SWITCH_PUSH, U1 ProMicro

Commit message: component placement
Connections:
- net at SW30.2: now also D30.1 (A)
Changed lines of the file:
@@
 LIBS:component
 LIBS:ProMicro
+LIBS:ErgoDOX-cache
 EELAYER 25 0
 EELAYER END
@@
 Connection ~ 6400 7350
 Connection ~ 6400 8000
+Wire Wire Line
+	5700 6050 5700 6150
+Wire Wire Line
+	5700 6150 5600 6150
 $EndSCHEMATC

Commit message: component placement circuit mod
replicated the Let's split cirucit design to this project. finilized placement of the initial components
Parts:
- added J5, J6: JMP, BishopKicadConsolidated:SOLDER_JUMPER_3, symbol 3PIN
- added SW45, SW46: SWITCH_PUSH, BishopKicadConsolidated:SOLDER_JUMPER_2, symbol SWITCH_PUSH
- added W1, W2, W3, W4, W5: TEST_1P, BishopKicadConsolidated:PIN_1, symbol TEST_1P
Connections:
- net COL0: now also U1.6 (PF5); no longer U1.5 (PF4)
- net COL1: now also U1.7 (PF6); no longer U1.6 (PF5)
- net COL2: now also U1.8 (PF7); no longer U1.7 (PF6)
- net COL3: now also U1.9 (PB1); no longer U1.8 (PF7)
- net COL4: now also U1.10 (PB3); no longer U1.9 (PB1)
- net COL5: now also U1.11 (PB2); no longer U1.10 (PB3)
- net COL6: now also U1.12 (PB6); no longer U1.11 (PB2)
- net GND: now also J3.1, J4.1, J5.1, J6.1, SW45.0 (GND), SW45.2, SW46.0 (GND), SW46.2; no longer J3.3, J4.3
- net LED_A: no longer U1.12 (PB6)
- net LED_B: no longer U1.18 (PD0)
- net LED_C: no longer U1.17 (PD1)
- net VCC: now also J3.3, J4.3, J5.3, J6.3; no longer J3.1, J4.1
- net at J2.1, J3.2: now also J5.2
- net at J2.4, J4.2: now also J6.2
- net at U1.3 (RST): now also SW45.1, SW46.1
- net SCLM renamed XTRADATA
- net XTRADATA: now also U1.17 (PD1), W1.1, W2.1; no longer U1.13 (PD3)
- net SDAM renamed DATA
- net DATA: now also U1.18 (PD0); no longer R1.2, U1.14 (PD2)
- new net: U1.13 (PD3), W3.1
- new net: U1.14 (PD2), W4.1
- new net: U1.5 (PF4), W5.1
Other:
- moved on the sheet: J1, J2, J3, J4, LED_A1, LED_B1, LED_C1, R1, R2, RA1, RB1, RC1
