File: _autosave-ErgoDOX.kicad_pcb (KiCad board)
At the start: 2 copper layers, 182.8 x 158.9 mm, 113 parts, among them J1 USB, J2 3.5mm, J3 JMP, J4 JMP, J5 JMP, J6 JMP, SW1 SWITCH_PUSH, SW10 SWITCH_PUSH, SW11 SWITCH_PUSH, SW12 SWITCH_PUSH, SW13 SWITCH_PUSH, SW14 SWITCH_PUSH, SW15 SWITCH_PUSH, SW16 SWITCH_PUSH, SW17 SWITCH_PUSH, SW18 SWITCH_PUSH, SW19 SWITCH_PUSH, SW2 SWITCH_PUSH, SW20 SWITCH_PUSH, SW21 SWITCH_PUSH, SW22 SWITCH_PUSH, SW23 SWITCH_PUSH, SW24 SWITCH_PUSH, SW25 SWITCH_PUSH, SW26 SWITCH_PUSH, SW27 SWITCH_PUSH, SW28 SWITCH_PUSH, SW29 SWITCH_PUSH, SW3 SWITCH_PUSH, SW30 SWITCH_PUSH, SW31 SWITCH_PUSH, SW32 SWITCH_PUSH, SW33 SWITCH_PUSH, SW34 SWITCH_PUSH, SW35 SWITCH_PUSH, SW36 SWITCH_PUSH, SW37 SWITCH_PUSH, SW38 SWITCH_PUSH, SW39 SWITCH_PUSH, SW4 SWITCH_PUSH, SW40 SWITCH_PUSH, SW41 SWITCH_PUSH, SW42 SWITCH_PUSH, SW43 SWITCH_PUSH, SW44 SWITCH_PUSH, SW45 SWITCH_PUSH, SW46 SWITCH_PUSH, SW5 SWITCH_PUSH, SW6 SWITCH_PUSH, SW7 SWITCH_PUSH, SW8 SWITCH_PUSH, SW9 SWITCH_PUSH, U1 ProMicro

Commit message: autosave
Other:
- board text added: "ErgoDox 2.0"
Changed lines of the file:
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@@
     (area 22.890479 30.289499 206.108301 189.542421)
     (thickness 1.6002)
-    (drawings 33)
+    (drawings 34)
     (tracks 0)
     (zones 0)
@@
       (xy -2.939146 -5.117164)) (layer F.SilkS) (width 0.01))
   )
+  (gr_text "ErgoDox 2.0" (at 90.678 51.816) (layer F.SilkS)
+    (effects (font (size 6 6) (thickness 1)))
+  )
   (gr_circle (center 139.065 91.567) (end 139.319 95.25) (layer Edge.Cuts) (width 0.381))
